File: AVR_programmer_debugger.kicad_pcb (KiCad board)
At the start: 2 copper layers, 66 x 19.4 mm, 22 parts, among them J1 Flipper Zero, J2 AVR-UPDI-6, J3 Conn_01x04, J4 AVR-ISP-10, SW1 SW_SPDT, U1 TXS0104EPWR, U2 TXS0104EPWR

Commit message: V1.2
Parts:
- added NT1: NetTie_2, NetTie:NetTie-2_SMD_Pad0.5mm, B.Cu at (139.0, 107.1)
- D1: value LED -> LED E6CC1206VGAC1UDA
- U1, U2: value TXS0104EPWR -> TXS0104ERGYR; footprint Package_SO:TSSOP-14_4.4x5mm_P0.65mm -> Package_DFN_QFN:Texas_S-PVQFN-N14_ThermalVias
- moved C1 5.08 mm to (139.3, 105.9)
- moved U2 1.31 mm to (140.8, 102.7)
- moved U1 0.64 mm to (99.0, 104.5), turned to 90 degrees
Connections:
- C1 pad 2: +3.3V -> /VCCA
- C3 pad 2: +3.3V -> /VCCA
- U1 pad 1: +3.3V -> /VCCA
- U1 pad 10: /~{RST}_s -> /MOSI_s
- U1 pad 11: /SCK_s -> /MISO_s
- U1 pad 12: /MOSI_s -> /SCK_s
- U1 pad 13: /MISO_s -> /~{RST}_s
- U1 pad 2: /MISO -> /~{RST}
- U1 pad 3: /MOSI -> /SCK
- U1 pad 4: /SCK -> /MISO
- U1 pad 5: /~{RST} -> /MOSI
- U1 pad 8: +3.3V -> /VCCA
- U2 pad 1: +3.3V -> /VCCA
- U2 pad 8: +3.3V -> /VCCA
Routing:
- net /VCCA: track 0.00 -> 70.4 mm, vias 0 -> 5
- net +3.3V: track 64.1 -> 22.1 mm, vias 2 -> 0
- net /VCCB: track 70.1 -> 77.1 mm
- net /RX: track 16.9 -> 23.1 mm, vias 0 -> 2
- net /SCK: track 7.77 -> 3.89 mm
- net /~{RST}: track 9.99 -> 6.48 mm
- net /MISO_s: track 13.1 -> 9.72 mm
- net /SCK_s: track 10.3 -> 7.46 mm
- net /TX: track 12.8 -> 15.6 mm, vias 1 -> 2
- net /UPDI_RX_s: track 18.0 -> 20.6 mm
- net /UPDI_TX_s: track 1.75 -> 4.30 mm
- net /~{RST}_s: track 8.62 -> 6.81 mm
- net /MISO: track 5.95 -> 4.21 mm
- net /UPDI_RX: track 10.5 -> 12.1 mm
- net /MOSI_s: track 11.1 -> 10.0 mm, vias 0 -> 1
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Other:
- board text added: "GZT, V 1.2, Mar. 2024"
- board text removed: "GZT, V 1.0, Sept. 2023"
